Commit message: working

File: plex_moveit/urdf/plex.urdf.xacro (robot description, xacro)
@@ -1,4 +1,4 @@
 <?xml version="1.0"?>
-<robot xmlns:xacro="http://www.ros.org/wiki/xacro" name="plex_arm_3">
+<robot xmlns:xacro="http://www.ros.org/wiki/xacro" name="plex">
   <!-- ================================================================
        Macros
@@ -14,5 +14,5 @@
         <origin xyz="0 0 0" rpy="0 0 0" />
         <geometry>
-          <mesh filename="package://plex_arm_urdf_3/meshes/${name}.STL" />
+          <mesh filename="package://plex_moveit/meshes/${name}.STL" />
         </geometry>
         <material name="">
@@ -23,5 +23,5 @@
         <origin xyz="0 0 0" rpy="0 0 0" />
         <geometry>
-          <mesh filename="package://plex_arm_urdf_3/meshes/${name}.STL" />
+          <mesh filename="package://plex_moveit/meshes/${name}.STL" />
         </geometry>
       </collision>
