Commit message: plex_moveit

File: plex_ethercat/description/config/motor_drive.config.xacro (robot description, xacro)
@@ -1,6 +1,6 @@
 <?xml version="1.0"?>
-<robot xmlns:xacro="http://www.ros.org/wiki/xacro" name="ethercat_zeroerr">
+<robot xmlns:xacro="http://www.ros.org/wiki/xacro" name="plex_ethercat">
   <link name="world"/>
-  <xacro:include filename="$(find ethercat_zeroerr)/description/ros2_control/motor_drive.ros2_control.xacro" />
-  <xacro:ethercat_zeroerr/>
+  <xacro:include filename="$(find plex_ethercat)/description/ros2_control/motor_drive.ros2_control.xacro" />
+  <xacro:plex_ethercat/>
 </robot>

File: plex_ethercat/description/ros2_control/motor_drive.ros2_control.xacro (robot description, xacro)
@@ -2,6 +2,6 @@
 <robot xmlns:xacro="http://www.ros.org/wiki/xacro">
   <!-- ZeroErr eRob 5-axis EtherCAT ros2_control description -->
-  <xacro:macro name="ethercat_zeroerr">
-    <ros2_control name="ethercat_zeroerr" type="system">
+  <xacro:macro name="plex_ethercat">
+    <ros2_control name="plex_ethercat" type="system">
       <hardware>
         <plugin>ethercat_driver/EthercatDriver</plugin>
@@ -29,5 +29,5 @@
           <param name="position">0</param>
           <param name="mode_of_operation">9</param>
-          <param name="slave_config">$(find ethercat_zeroerr)/config/zeroerr_config.yaml</param>
+          <param name="slave_config">$(find plex_ethercat)/config/zeroerr_config.yaml</param>
         </ec_module>
       </joint>
@@ -52,5 +52,5 @@
           <param name="position">1</param>
           <param name="mode_of_operation">9</param>
-          <param name="slave_config">$(find ethercat_zeroerr)/config/zeroerr_config.yaml</param>
+          <param name="slave_config">$(find plex_ethercat)/config/zeroerr_config.yaml</param>
         </ec_module>
       </joint>
@@ -75,5 +75,5 @@
           <param name="position">2</param>
           <param name="mode_of_operation">9</param>
-          <param name="slave_config">$(find ethercat_zeroerr)/config/zeroerr_config.yaml</param>
+          <param name="slave_config">$(find plex_ethercat)/config/zeroerr_config.yaml</param>
         </ec_module>
       </joint>
@@ -98,5 +98,5 @@
           <param name="position">3</param>
           <param name="mode_of_operation">9</param>
-          <param name="slave_config">$(find ethercat_zeroerr)/config/zeroerr_config.yaml</param>
+          <param name="slave_config">$(find plex_ethercat)/config/zeroerr_config.yaml</param>
         </ec_module>
       </joint>
@@ -121,5 +121,5 @@
           <param name="position">4</param>
           <param name="mode_of_operation">9</param>
-          <param name="slave_config">$(find ethercat_zeroerr)/config/zeroerr_config.yaml</param>
+          <param name="slave_config">$(find plex_ethercat)/config/zeroerr_config.yaml</param>
         </ec_module>
       </joint>
@@ -135,5 +135,5 @@
           <param name="alias">0</param>
           <param name="position">5</param>
-          <param name="slave_config">$(find ethercat_zeroerr)/config/stepper_config.yaml</param>
+          <param name="slave_config">$(find plex_ethercat)/config/stepper_config.yaml</param>
         </ec_module>
       </joint>

File: plex_moveit/config/plex_moevit.ros2_control.xacro (robot description, xacro)
@@ -1,5 +1,5 @@
 <?xml version="1.0"?>
 <robot xmlns:xacro="http://www.ros.org/wiki/xacro">
-    <xacro:macro name="plex_arm_urdf_3_ros2_control" params="name initial_positions_file">
+    <xacro:macro name="plex_moveit_ros2_control" params="name initial_positions_file">
         <xacro:property name="initial_positions" value="${load_yaml(initial_positions_file)['initial_positions']}"/>
         <ros2_control name="${name}" type="system">

Commit message: Integrate rover drive EtherCAT slaves

File: plex_ethercat/description/config/motor_drive.config.xacro (robot description, xacro)
@@ -2,5 +2,6 @@
 <robot xmlns:xacro="http://www.ros.org/wiki/xacro" name="plex_ethercat">
   <link name="world"/>
+  <xacro:arg name="use_drive" default="false"/>
   <xacro:include filename="$(find plex_ethercat)/description/ros2_control/motor_drive.ros2_control.xacro" />
-  <xacro:plex_ethercat/>
+  <xacro:plex_ethercat use_drive="$(arg use_drive)"/>
 </robot>

File: plex_ethercat/description/ros2_control/motor_drive.ros2_control.xacro (robot description, xacro)
@@ -1,6 +1,7 @@
 <?xml version="1.0"?>
 <robot xmlns:xacro="http://www.ros.org/wiki/xacro">
-  <!-- ZeroErr eRob 5-axis EtherCAT ros2_control description -->
-  <xacro:macro name="plex_ethercat">
+  <xacro:include filename="$(find spear_drive)/description/ros2_control/drive_interfaces.ros2_control.xacro"/>
+  <!-- Shared arm and rover EtherCAT master. Physical slave order is 0-15. -->
+  <xacro:macro name="plex_ethercat" params="use_drive:=false">
     <ros2_control name="plex_ethercat" type="system">
       <hardware>
@@ -138,4 +139,9 @@
         </ec_module>
       </joint>
+      <xacro:if value="${use_drive}">
+        <xacro:spear_drive_ethercat_joints
+          drive_slave_config="$(find spear_drive)/config/brushed_dc_config.yaml"
+          steering_slave_config="$(find plex_ethercat)/config/stepper_config.yaml"/>
+      </xacro:if>
     </ros2_control>
   </xacro:macro>

File: spear_drive/description/drive_mock.urdf.xacro (robot description, xacro)
@@ -41,6 +41,19 @@
     <xacro:macro name="mock_drive" params="joint">
       <joint name="${joint}">
-        <command_interface name="effort"/>
-        <state_interface name="velocity">
+        <command_interface name="current"/>
+        <command_interface name="control_word"/>
+        <state_interface name="status_word">
+          <param name="initial_value">4.0</param>
+        </state_interface>
+        <state_interface name="current">
+          <param name="initial_value">0.0</param>
+        </state_interface>
+        <state_interface name="encoder_counts_per_second">
+          <param name="initial_value">0.0</param>
+        </state_interface>
+        <state_interface name="encoder_counts">
+          <param name="initial_value">0.0</param>
+        </state_interface>
+        <state_interface name="duty_cycle">
           <param name="initial_value">0.0</param>
         </state_interface>

File: spear_drive/description/ros2_control/drive_interfaces.ros2_control.xacro (robot description, xacro)
@@ -4,7 +4,7 @@
     Call this macro inside the ONE existing master-0 ros2_control system after
     the arm joints. Running a second EtherCAT master for the drivetrain is not
-    supported. The two slave configuration paths must come from the embedded
-    team's final PDO descriptions; this package intentionally does not invent
-    vendor IDs, object indexes, data types, or scaling.
+    supported. The brushed-DC mapping is verified against the current embedded
+    repository; steering remains provisional until the flashed boards are
+    confirmed to match the arm stepper firmware.
   -->
   <xacro:macro name="spear_drive_ethercat_joints"
@@ -12,6 +12,11 @@
     <xacro:macro name="drive_slave" params="joint slave_position">
       <joint name="${joint}">
-        <command_interface name="effort"/>
-        <state_interface name="velocity"/>
+        <command_interface name="current"/>
+        <command_interface name="control_word"/>
+        <state_interface name="status_word"/>
+        <state_interface name="current"/>
+        <state_interface name="encoder_counts_per_second"/>
+        <state_interface name="encoder_counts"/>
+        <state_interface name="duty_cycle"/>
         <ec_module name="${joint}_ethercat">
           <plugin>ethercat_generic_plugins/GenericEcSlave</plugin>
@@ -24,6 +29,11 @@
     <xacro:macro name="steering_slave" params="joint slave_position">
       <joint name="${joint}">
+        <!-- The unused interfaces preserve the arm stepper's fixed PDO map. -->
+        <command_interface name="control_word"/>
         <command_interface name="position"/>
+        <command_interface name="velocity"/>
+        <state_interface name="status_word"/>
         <state_interface name="position"/>
+        <state_interface name="velocity"/>
         <ec_module name="${joint}_ethercat">
           <plugin>ethercat_generic_plugins/GenericEcSlave</plugin>
