Commit message: dc motor

File: plex_ethercat/description/ros2_control/motor_drive.ros2_control.xacro (robot description, xacro)
@@ -9,5 +9,5 @@
         <param name="control_frequency">1000</param>
       </hardware>
-      <joint name="joint_1">
+      <!-- <joint name="joint_1">
         <state_interface name="position"/>
         <state_interface name="velocity"/>
@@ -137,4 +137,18 @@
           <param name="slave_config">$(find plex_ethercat)/config/stepper_config.yaml</param>
         </ec_module>
+      </joint> -->
+      <joint name="drive_1">
+        <command_interface name="control_word"/>
+        <command_interface name="position"/>
+        <command_interface name="velocity"/>
+        <state_interface name="status_word"/>
+        <state_interface name="position"/>
+        <state_interface name="velocity"/>
+        <ec_module name="Stepper_joint_6">
+          <plugin>ethercat_generic_plugins/GenericEcSlave</plugin>
+          <param name="alias">0</param>
+          <param name="position">0</param>
+          <param name="slave_config">$(find plex_ethercat)/config/dc_config.yaml</param>
+        </ec_module>
       </joint>
     </ros2_control>
