Commit message: dc motor

File: plex_ethercat/description/ros2_control/motor_drive.ros2_control copy 2.xacro (robot description, xacro)
@@ -9,5 +9,5 @@
         <param name="control_frequency">1000</param>
       </hardware>
-      <!-- <joint name="joint_1">
+      <joint name="joint_1">
         <state_interface name="position"/>
         <state_interface name="velocity"/>
@@ -137,6 +137,6 @@
           <param name="slave_config">$(find plex_ethercat)/config/stepper_config.yaml</param>
         </ec_module>
-      </joint> -->
-      <joint name="drive_1">
+      </joint>
+      <!-- <joint name="drive_1">
         <command_interface name="control_word"/>
         <command_interface name="position"/>
@@ -150,40 +150,8 @@
           <plugin>ethercat_generic_plugins/GenericEcSlave</plugin>
           <param name="alias">0</param>
-          <param name="position">1</param>
+          <param name="position">0</param>
           <param name="slave_config">$(find plex_ethercat)/config/dc_config.yaml</param>
         </ec_module>
-      </joint>
-      <joint name="drive_2">
-        <command_interface name="control_word"/>
-        <command_interface name="position"/>
-        <command_interface name="velocity"/>
-        <command_interface name="current"/>
-        <state_interface name="status_word"/>
-        <state_interface name="position"/>
-        <state_interface name="velocity"/>
-        <state_interface name="current"/>
-        <ec_module name="drive_joint_2">
-          <plugin>ethercat_generic_plugins/GenericEcSlave</plugin>
-          <param name="alias">0</param>
-          <param name="position">2</param>
-          <param name="slave_config">$(find plex_ethercat)/config/dc_config.yaml</param>
-        </ec_module>
-      </joint>
-      <joint name="drive_3">
-        <command_interface name="control_word"/>
-        <command_interface name="position"/>
-        <command_interface name="velocity"/>
-        <command_interface name="current"/>
-        <state_interface name="status_word"/>
-        <state_interface name="position"/>
-        <state_interface name="velocity"/>
-        <state_interface name="current"/>
-        <ec_module name="drive_joint_3">
-          <plugin>ethercat_generic_plugins/GenericEcSlave</plugin>
-          <param name="alias">0</param>
-          <param name="position">3</param>
-          <param name="slave_config">$(find plex_ethercat)/config/dc_config.yaml</param>
-        </ec_module>
-      </joint>
+      </joint> -->
     </ros2_control>
   </xacro:macro>

File: plex_ethercat/description/ros2_control/motor_drive.ros2_control copy.xacro (robot description, xacro)
@@ -150,37 +150,5 @@
           <plugin>ethercat_generic_plugins/GenericEcSlave</plugin>
           <param name="alias">0</param>
-          <param name="position">1</param>
-          <param name="slave_config">$(find plex_ethercat)/config/dc_config.yaml</param>
-        </ec_module>
-      </joint>
-      <joint name="drive_2">
-        <command_interface name="control_word"/>
-        <command_interface name="position"/>
-        <command_interface name="velocity"/>
-        <command_interface name="current"/>
-        <state_interface name="status_word"/>
-        <state_interface name="position"/>
-        <state_interface name="velocity"/>
-        <state_interface name="current"/>
-        <ec_module name="drive_joint_2">
-          <plugin>ethercat_generic_plugins/GenericEcSlave</plugin>
-          <param name="alias">0</param>
-          <param name="position">2</param>
-          <param name="slave_config">$(find plex_ethercat)/config/dc_config.yaml</param>
-        </ec_module>
-      </joint>
-      <joint name="drive_3">
-        <command_interface name="control_word"/>
-        <command_interface name="position"/>
-        <command_interface name="velocity"/>
-        <command_interface name="current"/>
-        <state_interface name="status_word"/>
-        <state_interface name="position"/>
-        <state_interface name="velocity"/>
-        <state_interface name="current"/>
-        <ec_module name="drive_joint_3">
-          <plugin>ethercat_generic_plugins/GenericEcSlave</plugin>
-          <param name="alias">0</param>
-          <param name="position">3</param>
+          <param name="position">0</param>
           <param name="slave_config">$(find plex_ethercat)/config/dc_config.yaml</param>
         </ec_module>
