Commit message: ros2 control

File: plex_ethercat/description/ros2_control/motor_drive_2.ros2_control.xacro (robot description, xacro)
@@ -139,4 +139,22 @@
         </ec_module>
       </joint>
+    <!--.........................gripper.............................-->
+      <joint name="gripper">
+        <command_interface name="control_word"/>
+        <command_interface name="position"/>
+        <command_interface name="velocity"/>
+        <command_interface name="current"/>
+        <state_interface name="status_word"/>
+        <state_interface name="position"/>
+        <state_interface name="velocity"/>
+        <state_interface name="current"/>
+        <ec_module name="gripper_1">
+          <plugin>ethercat_generic_plugins/GenericEcSlave</plugin>
+          <param name="alias">0</param>
+          <param name="position">0</param>
+          <param name="slave_config">$(find plex_ethercat)/config/dc_config.yaml</param>
+        </ec_module>
+      </joint>
+    </ros2_control>
     <!--.........................drive.............................-->
       <joint name="wheel_front_left_joint">
@@ -144,7 +162,9 @@
         <command_interface name="position"/>
         <command_interface name="velocity"/>
-        <state_interface name="status_word"/>
-        <state_interface name="position"/>
-        <state_interface name="velocity"/>
+        <command_interface name="current"/>
+        <state_interface name="status_word"/>
+        <state_interface name="position"/>
+        <state_interface name="velocity"/>
+        <state_interface name="current"/>
         <ec_module name="motor_1">
           <plugin>ethercat_generic_plugins/GenericEcSlave</plugin>
@@ -159,7 +179,9 @@
         <command_interface name="position"/>
         <command_interface name="velocity"/>
-        <state_interface name="status_word"/>
-        <state_interface name="position"/>
-        <state_interface name="velocity"/>
+        <command_interface name="current"/>
+        <state_interface name="status_word"/>
+        <state_interface name="position"/>
+        <state_interface name="velocity"/>
+        <state_interface name="current"/>
         <ec_module name="motor_2">
           <plugin>ethercat_generic_plugins/GenericEcSlave</plugin>
@@ -174,7 +196,9 @@
         <command_interface name="position"/>
         <command_interface name="velocity"/>
-        <state_interface name="status_word"/>
-        <state_interface name="position"/>
-        <state_interface name="velocity"/>
+        <command_interface name="current"/>
+        <state_interface name="status_word"/>
+        <state_interface name="position"/>
+        <state_interface name="velocity"/>
+        <state_interface name="current"/>
         <ec_module name="motor_3">
           <plugin>ethercat_generic_plugins/GenericEcSlave</plugin>
@@ -189,7 +213,9 @@
         <command_interface name="position"/>
         <command_interface name="velocity"/>
-        <state_interface name="status_word"/>
-        <state_interface name="position"/>
-        <state_interface name="velocity"/>
+        <command_interface name="current"/>
+        <state_interface name="status_word"/>
+        <state_interface name="position"/>
+        <state_interface name="velocity"/>
+        <state_interface name="current"/>
         <ec_module name="motor_4">
           <plugin>ethercat_generic_plugins/GenericEcSlave</plugin>
@@ -204,7 +230,9 @@
         <command_interface name="position"/>
         <command_interface name="velocity"/>
-        <state_interface name="status_word"/>
-        <state_interface name="position"/>
-        <state_interface name="velocity"/>
+        <command_interface name="current"/>
+        <state_interface name="status_word"/>
+        <state_interface name="position"/>
+        <state_interface name="velocity"/>
+        <state_interface name="current"/>
         <ec_module name="motor_5">
           <plugin>ethercat_generic_plugins/GenericEcSlave</plugin>
@@ -219,7 +247,9 @@
         <command_interface name="position"/>
         <command_interface name="velocity"/>
-        <state_interface name="status_word"/>
-        <state_interface name="position"/>
-        <state_interface name="velocity"/>
+        <command_interface name="current"/>
+        <state_interface name="status_word"/>
+        <state_interface name="position"/>
+        <state_interface name="velocity"/>
+        <state_interface name="current"/>
         <ec_module name="motor_6">
           <plugin>ethercat_generic_plugins/GenericEcSlave</plugin>
@@ -241,5 +271,5 @@
           <param name="alias">0</param>
           <param name="position">0</param>
-          <param name="slave_config">$(find plex_ethercat)/config/dc_config.yaml</param>
+          <param name="slave_config">$(find plex_ethercat)/config/stepper_config.yaml</param>
         </ec_module>
       </joint>
@@ -255,5 +285,5 @@
           <param name="alias">0</param>
           <param name="position">0</param>
-          <param name="slave_config">$(find plex_ethercat)/config/dc_config.yaml</param>
+          <param name="slave_config">$(find plex_ethercat)/config/stepper_config.yaml</param>
         </ec_module>
       </joint>
@@ -269,5 +299,5 @@
           <param name="alias">0</param>
           <param name="position">0</param>
-          <param name="slave_config">$(find plex_ethercat)/config/dc_config.yaml</param>
+          <param name="slave_config">$(find plex_ethercat)/config/stepper_config.yaml</param>
         </ec_module>
       </joint>
@@ -283,5 +313,5 @@
           <param name="alias">0</param>
           <param name="position">0</param>
-          <param name="slave_config">$(find plex_ethercat)/config/dc_config.yaml</param>
+          <param name="slave_config">$(find plex_ethercat)/config/stepper_config.yaml</param>
         </ec_module>
       </joint>
